File: Hardware/FRReceiverProgPcb/FRReceiverProg.kicad_pcb (KiCad board)
At the start: 2 copper layers, 55.5 x 20.5 mm, 13 parts, among them J1 Conn_01x05, J2 Conn_02x04_Odd_Even, J3 Conn_02x05_Odd_Even, J4 Conn_01x02, J5 Conn_01x06, J6 Conn_01x02, J7 Conn_01x03, J8 Conn_01x05, J9 Conn_01x02, SW1 SW_Push

Commit message: support FRLVH board
Parts:
- added J10: Conn_02x04_Odd_Even, Connector_PinSocket_2.54mm:PinSocket_2x04_P2.54mm_Vertical, F.Cu at (96.5, 101.6)
- moved J2 12.0 mm to (101.5, 113.0)
- moved J3 5.40 mm to (147.0, 101.6)
- moved J6 2.05 mm to (139.0, 115.0)
- moved J8 1.27 mm to (108.0, 99.1)
- moved J9 1.27 mm to (105.4, 106.7)
Routing:
- net /CLK: track 71.8 -> 98.1 mm, vias 6 -> 4
- net /MOSI: track 75.9 -> 101.1 mm, vias 3 -> 6
- net /MISO: track 69.3 -> 90.0 mm, vias 7 -> 5
- net /RESET: track 72.7 -> 92.0 mm, vias 6 -> 8
- net /STX: track 41.8 -> 53.9 mm
- net /SRX: track 38.3 -> 50.3 mm
- net /VCC: track 129.0 -> 122.7 mm
Other:
- board size 55.5 x 20.5 mm -> 60 x 20.5 mm
- board text added: "FR- LVH"
- board text added: "FR-8/4"
- board text added: "V4"
- board text removed: "FR-8"
- board text removed: "USBASP"
